Commit message: URDF: diff-drive robot, launch file, castor height corrected

File: src/my_robot_description/urdf/robot.urdf (robot description, URDF)
Before this commit: robot my_robot, 4 links, 3 joints
Joints:
- joint castor_wheel_joint: origin xyz=0.12 0 -0.055 rpy=0 0 0 -> xyz=0.12 0 -0.0525 rpy=0 0 0
